File: Esquematico_2_k10/Esquematico_2_k10.kicad_sch (KiCad schematic)
At the start: 1 part

Commit message: Nueva carga de esquematicos y footprints
Parts:
- removed U?: QMC5883P, LGA-16_L3.0-W3.0-P0.50-BL_SQ, symbol Esquematico_2_k10-altium-import:root_0_QMC5883P_
- added U1: QMC5883P, QMC5883P:LGA-16_L3.0-W3.0-P0.50-BL_SQ, symbol Esquematico_2_k10-altium-import:root_0_QMC5883P_
Other:
- note removed: "Mira esto puto, este el esquematico del magnetonmetro y su footprint esta en la misma carpeta con el nombre se llama LGA-16_L3.0-W3.0-P0.50-BL_SQ el footprint"
Changed lines of the file:
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@@
 	(generator_version "10.0")
 	(paper "User" 124.46 99.06)
-	(text "Mira esto puto, este el esquematico del magnetonmetro y su footprint esta en la misma carpeta con el nombre\nse llama LGA-16_L3.0-W3.0-P0.50-BL_SQ el footprint"
-		(exclude_from_sim no)
-		(at 58.674 25.908 0)
-		(effects
-			(font
-				(size 1.27 1.27)
-			)
-		)
-	)
 	(symbol
 		(lib_id "Esquematico_2_k10-altium-import:root_0_QMC5883P_")
@@
 		(in_pos_files yes)
 		(dnp no)
-		(property "Reference" "U?"
+		(property "Reference" "U1"
 			(at 63.5 49.53 90)
 			(show_name no)
@@
 		)
 		(property "Value" "QMC5883P"
-			(at 58.42 63.246 90)
-			(show_name no)
-			(do_not_autoplace no)
-			(effects
-				(font
-					(size 1.27 1.27)
-				)
-				(justify right bottom)
-			)
-		)
-		(property "Footprint" "LGA-16_L3.0-W3.0-P0.50-BL_SQ"
+			(at 59.436 61.722 90)
+			(show_name no)
+			(do_not_autoplace no)
+			(effects
+				(font
+					(size 1.27 1.27)
+				)
+				(justify right bottom)
+			)
+		)
+		(property "Footprint" "QMC5883P:LGA-16_L3.0-W3.0-P0.50-BL_SQ"
 			(at 63.5 49.53 0)
 			(hide yes)
@@
 			)
 		)
+		(pin "1"
+		)
 		(pin "3"
 		)
+		(pin "6"
+		)
+		(pin "8"
+		)
+		(pin "5"
+		)
 		(pin "2"
 		)
-		(pin "1"
+		(pin "4"
+		)
+		(pin "7"
+		)
+		(pin "9"
+		)
+		(pin "10"
+		)
+		(pin "11"
+		)
+		(pin "12"
 		)
 		(pin "13"
 		)
-		(pin "7"
+		(pin "14"
+		)
+		(pin "15"
 		)
 		(pin "16"
-		)
-		(pin "10"
-		)
-		(pin "6"
-		)
-		(pin "12"
-		)
-		(pin "11"
-		)
-		(pin "14"
-		)
-		(pin "15"
-		)
-		(pin "4"
-		)
-		(pin "9"
-		)
-		(pin "8"
-		)
-		(pin "5"
 		)
 		(instances
 			(project ""
-				(path "/fd9e1921-b3d8-4302-87f4-eaf394000729"
-					(reference "U?")
+				(path "/8bd3707c-b4ed-4787-a9b1-9d02c6aeb16b"
+					(reference "U1")
 					(unit 1)
 				)
