File: Esquematico_1/_autosave-microcontrolador.kicad_sch (KiCad schematic)
At the start: 13 parts, among them SW1 RST, SW2 BOOT, U2 STM32F405RGTx

Commit message: Update esquematico
Parts:
- removed C5: 4.7u, symbol Device:C
- removed C6: 100n, symbol Device:C
- added C7: 10u, symbol Device:C
- added C8: 100n, symbol Device:C
- added FB1: FerriteBead, symbol Device:FerriteBead
Connections:
- net 3V3: now also FB1.1; no longer CARD1.4 (VDD)
- net GND: now also C7.1, C8.1
- net 3V3A: now reaches U2.13 (VDDA)
- net 3V3A: now also CARD1.4 (VDD), C7.2, C8.2, FB1.2
Other:
- moved on the sheet: U2, USB1
