File: Esquematico_1/sensores_.kicad_sch (KiCad schematic)
At the start: 10 parts, among them IC1 MAX-M10M-00B, U1 ICM-42688-P, U3 Mag, U4 BMP388

Commit message: Imu
Parts:
- added C10: 2.2 uF, symbol Device:C
- added C11: 0.1 uF, symbol Device:C
- added C9: 10 nF, symbol Device:C
Connections:
- net GND: now also U1.11 (RESV_11), U1.6 (GND), U1.7 (RESV_7), C10.2, C11.2, C9.2
- net SD0_IMU: now reaches U1.1 (AP_SDO/AP_AD0)
- net AP_CS_IMU: now reaches U1.12 (AP_CS)
- net CLK_IMU: now reaches U1.13 (AP_SCL/AP_SCLK)
- net SDIO_IMU: now reaches U1.14 (AP_SDA/AP_SDIO/AP_SDI)
- net INT1_IMU: now reaches U1.4 (INT1/INT)
- net +3.3V: now reaches U1.5 (VDDIO)
- net +3.3V: now also U1.8 (VDD), C10.1, C11.1, C9.1
- net INT2_IMU: now reaches U1.9 (INT2/FSYNC/CLKIN)
- no-connect marks 0 -> 3
Other:
- moved on the sheet: IC1, U1

Commit message: Update
Connections:
- net SCK1 renamed SCK_MAG
- net SDA1 renamed SDA_MAG
- net SP1_CS1 renamed CS_BM
- net SP1_INT renamed INT_BM
- net SP1_MOSI renamed MOSI_BM
- net SP1_SCK renamed SCK_BM
- net SPI1_MISO renamed MISO_BM
Other:
- moved on the sheet: C1, C4

Commit message: Correciones de tags
Connections:
- net +3.3V: now also C1.1, C3.1, C4.1, R1.1, R2.1, U4.1 (VDDIO), U4.10 (VDD)
- net 3V3: no longer C1.1, C3.1, C4.1, R1.1, R2.1, U4.1 (VDDIO), U4.10 (VDD)
Other:
- moved on the sheet: IC1
