File: Esquematico_1/sensores_.kicad_sch (KiCad schematic)
At the start: 11 parts, among them U3 LSM6DSV16XTR, U4 BMP388, U7 MMC5983MA

Commit message: feature cambio de stackup, cambio de ruteo del IMU
Connections:
- net MISO_IMU: now also U3.1 (SDO/SA0); no longer U3.14 (SDA)
- net MOSI_IMU: now also U3.14 (SDA); no longer U3.1 (SDO/SA0)
