File: Esquematico_1/power.kicad_sch (KiCad schematic)
At the start: 22 parts, among them IC1 AP2112K-3.3TRG1, U6 TPS54302DDCR

Commit message: Cambios de Diodos
Parts:
- D1, D4: footprint Package_TO_SOT_SMD:SOT-23 -> Diode_SMD:D_SOD-323_HandSoldering
Changed lines of the file:
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@@
 			)
 		)
-		(property "Footprint" "Package_TO_SOT_SMD:SOT-23"
+		(property "Footprint" "Diode_SMD:D_SOD-323_HandSoldering"
 			(at 158.75 33.02 0)
 			(effects
@@
 			)
 		)
-		(property "Footprint" "Package_TO_SOT_SMD:SOT-23"
+		(property "Footprint" "Diode_SMD:D_SOD-323_HandSoldering"
 			(at 80.01 148.59 0)
 			(effects

Commit message: Cambio de IMU, creación del BOM
Parts:
- C12: LCSC Part Name (none) -> C113832
- C13, C15: value 0.1uF -> 100nF; LCSC Part Name (none) -> C1711
- C14: LCSC Part Name (none) -> C237493
- C16, C17: LCSC Part Name (none) -> C907991
- C18, C19: LCSC Part Name (none) -> C28323
- C33: LCSC Part Name (none) -> C1711
- D1, D4: LCSC Part Name (none) -> C124187
- F1: LCSC Part Name (none) -> C210838
- IC1: LCSC Part Name (none) -> C51118
- L1: now left out of the parts list
- R10: LCSC Part Name (none) -> C3000727
- R11: LCSC Part Name (none) -> C2933455
- R12: value 100K -> 100k; LCSC Part Name (none) -> C149504
- R13: LCSC Part Name (none) -> C2930408
- R17: LCSC Part Name (none) -> C149504
- R18: LCSC Part Name (none) -> C2930170
- R9: LCSC Part Name (none) -> C5159719
- U6: LCSC Part Name (none) -> C311983
