File: Esquematico_1/microcontrolador.kicad_sch (KiCad schematic)
At the start: 37 parts, among them U2 STM32F405RGTx

Commit message: Change Sd for Memory SPIO NAND
Parts:
- removed C30, C31: 12pF, Capacitor_SMD:C_0603_1608Metric_Pad1.08x0.95mm_HandSolder, symbol Device:C
- removed C34: 10uF, Capacitor_SMD:C_0603_1608Metric_Pad1.08x0.95mm_HandSolder, symbol Device:C
- removed C35: 100nF, Capacitor_SMD:C_0603_1608Metric_Pad1.08x0.95mm_HandSolder, symbol Device:C
- removed CARD1: MICRO SD, MOLEX 5033981892:TF-SMD_503398-1892, symbol 503398-1892:503398-1892
- removed LSE1: Crystal, ndx32khz:XTAL_NX3215SA_NDK, symbol Device:Crystal
- removed R3: 100k, Resistor_SMD:R_0805_2012Metric_Pad1.20x1.40mm_HandSolder, symbol Device:R
- removed R4, R5, R6, R7, R8: 47K, Resistor_SMD:R_0805_2012Metric_Pad1.20x1.40mm_HandSolder, symbol Device:R
- added U8: W25Q128JVSIQ, W25Q128JVSIQ:SOIC_128JVSIQ_WIN, symbol W25Q128JVSIQ:W25Q128JVSIQ
- C24: footprint Capacitor_SMD:C_0805_2012Metric_Pad1.18x1.45mm_HandSolder -> Capacitor_SMD:C_0603_1608Metric_Pad1.08x0.95mm_HandSolder
Connections:
- net CardDetect: no longer names the net of U2.56 (PB4)
- net LSE_IN: no longer names the net of U2.3 (PC14)
- net LSE_OUT: no longer names the net of U2.4 (PC15)
- net SDIO_CLK renamed Flash_MOSI
- net SDIO_D0: no longer names the net of U2.39 (PC8)
- net SDIO_D1: no longer names the net of U2.40 (PC9)
- net SDIO_D2 renamed Flash_SCK
- net SDIO_D3 renamed Flash_MISO
- no-connect marks 7 -> 9

Commit message: minor changes
Connections:
- net +3V3: now also U8.8 (VCC)
- net GND: now also U8.4 (GND)
Changed lines of the file:
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@@
 	(wire
 		(pts
+			(xy 200.66 48.26) (xy 200.66 52.07)
+		)
+		(stroke
+			(width 0)
+			(type default)
+		)
+	)
+	(wire
+		(pts
 			(xy 137.16 166.37) (xy 137.16 168.91)
 		)
@@
 	(wire
 		(pts
+			(xy 256.54 40.64) (xy 261.62 40.64)
+		)
+		(stroke
+			(width 0)
+			(type default)
+		)
+	)
+	(wire
+		(pts
 			(xy 76.2 119.38) (xy 76.2 121.92)
 		)
@@
 	(wire
 		(pts
+			(xy 203.2 48.26) (xy 200.66 48.26)
+		)
+		(stroke
+			(width 0)
+			(type default)
+		)
+	)
+	(wire
+		(pts
 			(xy 97.79 161.29) (xy 106.68 161.29)
 		)
@@
 	(wire
 		(pts
+			(xy 261.62 40.64) (xy 261.62 38.1)
+		)
+		(stroke
+			(width 0)
+			(type default)
+		)
+	)
+	(wire
+		(pts
 			(xy 148.59 154.94) (xy 148.59 158.75)
 		)
@@
 	)
 	(symbol
+		(lib_id "power:+3V3")
+		(at 261.62 38.1 0)
+		(unit 1)
+		(exclude_from_sim no)
+		(in_bom yes)
+		(on_board yes)
+		(dnp no)
+		(fields_autoplaced yes)
+		(property "Reference" "#PWR010"
+			(at 261.62 41.91 0)
+			(effects
+				(font
+					(size 1.27 1.27)
+				)
+				(hide yes)
+			)
+		)
+		(property "Value" "+3V3"
+			(at 261.62 33.02 0)
+			(effects
+				(font
+					(size 1.27 1.27)
+				)
+			)
+		)
+		(property "Footprint" ""
+			(at 261.62 38.1 0)
+			(effects
+				(font
+					(size 1.27 1.27)
+				)
+				(hide yes)
+			)
+		)
+		(property "Datasheet" ""
+			(at 261.62 38.1 0)
+			(effects
+				(font
+					(size 1.27 1.27)
+				)
+				(hide yes)
+			)
+		)
+		(property "Description" "Power symbol creates a global label with name \"+3V3\""
+			(at 261.62 38.1 0)
+			(effects
+				(font
+					(size 1.27 1.27)
+				)
+				(hide yes)
+			)
+		)
+		(pin "1"
+		)
+		(instances
+			(project "Esquematico_1"
+				(path "/de2d80c1-c21c-478d-b724-17659b714c38/65191e46-6d87-4ab8-a02b-a5dd631b354a"
+					(reference "#PWR010")
+					(unit 1)
+				)
+			)
+		)
+	)
+	(symbol
 		(lib_id "Device:R")
 		(at 137.16 162.56 0)
@@
 					(unit 1)
 				)
+			)
+		)
+	)
+	(symbol
+		(lib_id "power:GND")
+		(at 200.66 52.07 0)
+		(unit 1)
+		(exclude_from_sim no)
+		(in_bom yes)
+		(on_board yes)
+		(dnp no)
+		(fields_autoplaced yes)
+		(property "Reference" "#PWR09"
+			(at 200.66 58.42 0)
+			(effects
+				(font
+					(size 1.27 1.27)
+				)
+				(hide yes)
+			)
+		)
+		(property "Value" "GND"
+			(at 200.66 57.15 0)
+			(effects
+				(font
+					(size 1.27 1.27)
+				)
+			)
+		)
+		(property "Footprint" ""
+			(at 200.66 52.07 0)
+			(effects
+				(font
+					(size 1.27 1.27)
+				)
+				(hide yes)
+			)
+		)
+		(property "Datasheet" ""
+			(at 200.66 52.07 0)
+			(effects
+				(font
+					(size 1.27 1.27)
+				)
+				(hide yes)
+			)
+		)
+		(property "Description" "Power symbol creates a global label with name \"GND\" , ground"
+			(at 200.66 52.07 0)
+			(effects
+				(font
+					(size 1.27 1.27)
+				)
+				(hide yes)
+			)
+		)
+		(pin "1"
+		)
+		(instances
+			(project "Esquematico_1"
+				(path "/de2d80c1-c21c-478d-b724-17659b714c38/65191e46-6d87-4ab8-a02b-a5dd631b354a"
+					(reference "#PWR09")
+					(unit 1)
+				)

Commit message: Finishing Flash schematic
Parts:
- added R1, R2: 10k, symbol Device:R
Connections:
- net SDIO_CMD is gone; now on net Flash_CS: U2.54 (PD2)
- net +3V3: now also R1.1, R2.2
- net Flash_MISO: now also U8.2 (DO_(IO1))
- net Flash_MOSI: now also U8.5 (DI_(IO0))
- net Flash_SCK: now also U8.6 (CLK)
- net Flash_CS: now reaches U8.1 (/CS)
- net at U8.3: now also R2.1
- net at U8.7 (/HOLD_or_/RESET_(IO3)): now also R1.2
Other:
- note removed: "Esto es opcional, si se conecta al stm32 es una formaque te diga si hay una tarjeta insertada. pero no es necesario"

Commit message: Add: Dos bucks :(
Parts:
- R1, R2: footprint (none) -> Resistor_SMD:R_0805_2012Metric_Pad1.20x1.40mm_HandSolder
Connections:
- net Flash_MISO renamed MISO_Flash
- net Flash_MOSI renamed MOSI_Flash
- net Flash_SCK renamed CLK_Flash
Changed lines of the file:
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@@
 		)
 	)
-	(global_label "Flash_MOSI"
+	(global_label "MOSI_Flash"
 		(shape input)
 		(at 261.62 48.26 0)
@@
 		)
 	)
-	(global_label "Flash_SCK"
+	(global_label "CLK_Flash"
 		(shape input)
 		(at 261.62 45.72 0)
@@
 		)
 		(property "Intersheetrefs" "${INTERSHEET_REFS}"
-			(at 274.4022 45.72 0)
+			(at 274.2208 45.72 0)
 			(effects
 				(font
@@
 		)
 	)
+	(global_label "MOSI_Flash"
+		(shape input)
+		(at 88.9 95.25 180)
+		(fields_autoplaced yes)
+		(effects
+			(font
+				(size 1.27 1.27)
+			)
+			(justify right)
+		)
+		(property "Intersheetrefs" "${INTERSHEET_REFS}"
+			(at 75.2711 95.25 0)
+			(effects
+				(font
+					(size 1.27 1.27)
+				)
+				(justify right)
+				(hide yes)
+			)
+		)
+	)
 	(global_label "CLK_IMU"
 		(shape input)
@@
 		)
 	)
+	(global_label "CLK_Flash"
+		(shape input)
+		(at 88.9 90.17 180)
+		(fields_autoplaced yes)
+		(effects
+			(font
+				(size 1.27 1.27)
+			)
+			(justify right)
+		)
+		(property "Intersheetrefs" "${INTERSHEET_REFS}"
+			(at 76.2992 90.17 0)
+			(effects
+				(font
+					(size 1.27 1.27)
+				)
+				(justify right)
+				(hide yes)
+			)
+		)
+	)
 	(global_label "MOSI_IMU"
 		(shape output)
@@
 		)
 	)
-	(global_label "AP_CS_IMU"
+	(global_label "MISO_Flash"
 		(shape input)
-		(at 88.9 77.47 180)
+		(at 88.9 92.71 180)
 		(fields_autoplaced yes)
 		(effects
@@
 		)
 		(property "Intersheetrefs" "${INTERSHEET_REFS}"
-			(at 75.7548 77.47 0)
+			(at 75.2711 92.71 0)
 			(effects
 				(font
@@
 		)
 	)
-	(global_label "ESC4"
+	(global_label "AP_CS_IMU"
 		(shape input)
-		(at 140.97 49.53 0)
+		(at 88.9 77.47 180)
 		(fields_autoplaced yes)
 		(effects
@@
 				(size 1.27 1.27)
 			)
-			(justify left)
+			(justify right)
 		)
 		(property "Intersheetrefs" "${INTERSHEET_REFS}"
-			(at 148.7932 49.53 0)
+			(at 75.7548 77.47 0)
 			(effects
 				(font
 					(size 1.27 1.27)
 				)
-				(justify left)
+				(justify right)
 				(hide yes)
 			)
 		)
 	)
-	(global_label "Flash_MISO"
+	(global_label "ESC4"
 		(shape input)
-		(at 200.66 43.18 180)
+		(at 140.97 49.53 0)
 		(fields_autoplaced yes)
 		(effects
@@
 				(size 1.27 1.27)
 			)
-			(justify right)
+			(justify left)
 		)
 		(property "Intersheetrefs" "${INTERSHEET_REFS}"
-			(at 187.0311 43.18 0)
+			(at 148.7932 49.53 0)
 			(effects
 				(font
 					(size 1.27 1.27)
 				)
-				(justify right)
+				(justify left)
 				(hide yes)
 			)
 		)
 	)
-	(global_label "Flash_MOSI"
+	(global_label "MISO_Flash"
 		(shape input)
-		(at 88.9 95.25 180)
+		(at 200.66 43.18 180)
 		(fields_autoplaced yes)
 		(effects
@@
 		)
 		(property "Intersheetrefs" "${INTERSHEET_REFS}"
-			(at 75.2711 95.25 0)
+			(at 187.0311 43.18 0)
 			(effects
 				(font
@@
 		)
 	)
-	(global_label "Flash_SCK"
-		(shape input)
-		(at 88.9 90.17 180)
-		(fields_autoplaced yes)
-		(effects
-			(font
-				(size 1.27 1.27)
-			)
-			(justify right)
-		)
-		(property "Intersheetrefs" "${INTERSHEET_REFS}"
-			(at 76.1178 90.17 0)
-			(effects
-				(font
-					(size 1.27 1.27)
-				)
-				(justify right)
-				(hide yes)
-			)
-		)
-	)
 	(global_label "TELEM_ESC"
 		(shape input)
@@
 		)
 	)
-	(global_label "Flash_MISO"
-		(shape input)
-		(at 88.9 92.71 180)
-		(fields_autoplaced yes)
-		(effects
-			(font
-				(size 1.27 1.27)
-			)
-			(justify right)
-		)
-		(property "Intersheetrefs" "${INTERSHEET_REFS}"
-			(at 75.2711 92.71 0)
-			(effects
-				(font
-					(size 1.27 1.27)
-				)
-				(justify right)
-				(hide yes)
-			)
-		)
-	)
 	(global_label "SWDIO"
 		(shape bidirectional)
@@
 			)
 		)
-		(property "Footprint" ""
+		(property "Footprint" "Resistor_SMD:R_0805_2012Metric_Pad1.20x1.40mm_HandSolder"
 			(at 183.642 41.91 90)
 			(effects
@@
 			)
 		)
-		(property "Footprint" ""
+		(property "Footprint" "Resistor_SMD:R_0805_2012Metric_Pad1.20x1.40mm_HandSolder"
 			(at 263.652 38.1 90)
 			(effects
