File: hardware/esquematico/jst_cam.kicad_sch (KiCad schematic)
At the start: 16 parts, among them J1 Screw_Terminal_01x04, J2 Screw_Terminal_01x03, J3 Screw_Terminal_01x06, J4 Screw_Terminal_01x08, J5 SWD, J6 Screw_Terminal_01x04, J7 USB_C_Receptacle_USB2.0_16P, U5 USBLC6-2SC6

Commit message: chore(hardware): restore main PCB (SDIO microSD) to match current .ioc
The new PCB (W25Q128 SPI flash, TPSM bucks) now lives in the NewPCB branch.

Co-authored-by: Cursor <cursoragent@cursor.com>
Parts:
- added J8, J9: Screw_Terminal_01x01, TestPoint:TestPoint_Pad_2.5x2.5mm, symbol Connector:Screw_Terminal_01x01
- added JP1, JP2: SolderJumper_2_Open, Jumper:SolderJumper-2_P1.3mm_Open_RoundedPad1.0x1.5mm, symbol Jumper:SolderJumper_2_Open
Connections:
- net CRT: now also JP2.2 (B); no longer J4.6 (Pin_6)
- net ESC1: now also J4.1 (Pin_1); no longer J4.4 (Pin_4)
- net ESC2: now also J4.2 (Pin_2); no longer J4.3 (Pin_3)
- net ESC3: now also J4.3 (Pin_3); no longer J4.2 (Pin_2)
- net ESC4: now also J4.4 (Pin_4); no longer J4.1 (Pin_1)
- net GND: now also J4.8 (Pin_8), J9.1 (Pin_1); no longer J4.7 (Pin_7)
- net TELEM_ESC: now also J4.6 (Pin_6); no longer J4.5 (Pin_5)
- net VCC: now also JP1.2 (B); no longer J4.8 (Pin_8)
- new net: J4.7 (Pin_7), JP1.1 (A)
- new net: J4.5 (Pin_5), JP2.1 (A)
- new net Vbat: J8.1 (Pin_1)
Other:
- note added: "JST POWER"
