File: hardware/esquematico/microcontrolador.kicad_sch (KiCad schematic)
At the start: 28 parts, among them U2 STM32F405RGTx, U8 W25Q128JVSIQ

Commit message: chore(hardware): restore main PCB (SDIO microSD) to match current .ioc
The new PCB (W25Q128 SPI flash, TPSM bucks) now lives in the NewPCB branch.

Co-authored-by: Cursor <cursoragent@cursor.com>
Parts:
- removed R1, R2: 10k, Resistor_SMD:R_0805_2012Metric_Pad1.20x1.40mm_HandSolder, symbol Device:R
- removed U8: W25Q128JVSIQ, W25Q128JVSIQ:SOIC_128JVSIQ_WIN, symbol W25Q128JVSIQ:W25Q128JVSIQ
- added C30, C31: 12pF, Capacitor_SMD:C_0603_1608Metric_Pad1.08x0.95mm_HandSolder, symbol Device:C
- added C34: 10uF, Capacitor_SMD:C_0603_1608Metric_Pad1.08x0.95mm_HandSolder, symbol Device:C
- added C35: 100nF, Capacitor_SMD:C_0603_1608Metric_Pad1.08x0.95mm_HandSolder, symbol Device:C
- added CARD1: MICRO SD, MOLEX 5033981892:TF-SMD_503398-1892, symbol 503398-1892:503398-1892
- added LSE1: Crystal, ndx32khz:XTAL_NX3215SA_NDK, symbol Device:Crystal
- added R3: 100k, Resistor_SMD:R_0805_2012Metric_Pad1.20x1.40mm_HandSolder, symbol Device:R
- added R4, R5, R6, R7, R8: 47K, Resistor_SMD:R_0805_2012Metric_Pad1.20x1.40mm_HandSolder, symbol Device:R
- C24: footprint Capacitor_SMD:C_0603_1608Metric_Pad1.08x0.95mm_HandSolder -> Capacitor_SMD:C_0805_2012Metric_Pad1.18x1.45mm_HandSolder
Connections:
- net +3V3: now also C34.2, C35.2, CARD1.4 (VDD), R3.1, R4.1, R5.1, R6.1, R7.1, R8.1
- net GND: now also C30.2, C31.2, C34.1, C35.1, CARD1.10, CARD1.11 (EH), CARD1.6 (VSS)
- net LSE_IN: now reaches U2.3 (PC14)
- net LSE_IN: now also C31.1, LSE1.1
- net SDIO_D0: now reaches U2.39 (PC8)
- net SDIO_D0: now also CARD1.7 (DAT0), R7.2
- net LSE_OUT: now reaches U2.4 (PC15)
- net LSE_OUT: now also C30.1, LSE1.2
- net SDIO_D1: now reaches U2.40 (PC9)
- net SDIO_D1: now also CARD1.8 (DAT1), R8.2
- net CardDetect: now reaches U2.56 (PB4)
- net CardDetect: now also CARD1.9, R3.2
- net CLK_Flash renamed SDIO_D2
- net SDIO_D2: now also CARD1.1 (DAT2), R4.2
- net Flash_CS renamed SDIO_CMD
- net SDIO_CMD: now also CARD1.3 (CMD), R6.2
- net MISO_Flash renamed SDIO_D3
- net SDIO_D3: now also CARD1.2 (CD/DAT3), R5.2
- net MOSI_Flash renamed SDIO_CLK
- net SDIO_CLK: now also CARD1.5 (CLK)
- no-connect marks 9 -> 7
Other:
- note added: "Esto es opcional, si se conecta al stm32 es una formaque te diga si hay una tarjeta insertada. pero no es necesario"
