File: hardware/esquematico/sensores_.kicad_sch (KiCad schematic)
At the start: 11 parts, among them U3 LSM6DSV16XTR, U4 BMP388, U7 MMC5983MA

Commit message: chore(hardware): restore main PCB (SDIO microSD) to match current .ioc
The new PCB (W25Q128 SPI flash, TPSM bucks) now lives in the NewPCB branch.

Co-authored-by: Cursor <cursoragent@cursor.com>
Connections:
- net MISO_IMU: now also U3.14 (SDA); no longer U3.1 (SDO/SA0)
- net MOSI_IMU: now also U3.1 (SDO/SA0); no longer U3.14 (SDA)
Changed lines of the file:
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@@
-	(wire
-		(pts
-			(xy 38.1 26.67) (xy 40.64 26.67)
-		)
-		(stroke
-			(width 0)
-			(type default)
-		)
-	)
 	(wire
 		(pts
@@
 	(wire
 		(pts
+			(xy 106.68 26.67) (xy 111.76 26.67)
+		)
+		(stroke
+			(width 0)
+			(type default)
+		)
+	)
+	(wire
+		(pts
 			(xy 190.5 160.02) (xy 195.58 160.02)
 		)
@@
 	(wire
 		(pts
-			(xy 106.68 26.67) (xy 111.76 26.67)
-		)
-		(stroke
-			(width 0)
-			(type default)
-		)
-	)
-	(wire
-		(pts
 			(xy 40.64 30.48) (xy 40.64 31.75)
 		)
@@
 		(pts
 			(xy 40.64 39.37) (xy 40.64 41.91)
+		)
+		(stroke
+			(width 0)
+			(type default)
+		)
+	)
+	(wire
+		(pts
+			(xy 36.83 26.67) (xy 40.64 26.67)
 		)
 		(stroke
@@
 	(global_label "MISO_IMU"
 		(shape bidirectional)
-		(at 38.1 26.67 180)
-		(fields_autoplaced yes)
-		(effects
-			(font
-				(size 1.27 1.27)
-			)
-			(justify right)
-		)
-		(property "Intersheetrefs" "${INTERSHEET_REFS}"
-			(at 25.053 26.67 0)
-			(effects
-				(font
-					(size 1.27 1.27)
-				)
-				(justify right)
+		(at 111.76 26.67 0)
+		(fields_autoplaced yes)
+		(effects
+			(font
+				(size 1.27 1.27)
+			)
+			(justify left)
+		)
+		(property "Intersheetrefs" "${INTERSHEET_REFS}"
+			(at 124.807 26.67 0)
+			(effects
+				(font
+					(size 1.27 1.27)
+				)
+				(justify left)
 				(hide yes)
 			)
@@
 	(global_label "MOSI_IMU"
 		(shape output)
-		(at 111.76 26.67 0)
-		(fields_autoplaced yes)
-		(effects
-			(font
-				(size 1.27 1.27)
-			)
-			(justify left)
-		)
-		(property "Intersheetrefs" "${INTERSHEET_REFS}"
-			(at 123.6957 26.67 0)
-			(effects
-				(font
-					(size 1.27 1.27)
-				)
-				(justify left)
-				(hide yes)
-			)
+		(at 36.83 26.67 180)
+		(fields_autoplaced yes)
+		(effects
+			(font
+				(size 1.27 1.27)
+			)
+			(justify right)
+		)
+		(property "Intersheetrefs" "${INTERSHEET_REFS}"
+			(at 24.8943 26.67 0)
+			(effects
+				(font
+					(size 1.27 1.27)
+				)
+				(justify right)
+				(hide yes)
+			)
